File: PCB/DIYDSPv0.5/DIYDSPv0.5.kicad_pcb (KiCad board)
At the start: 4 copper layers, 100 x 100 mm, 292 parts, among them J1 Conn_01x03, J10 Conn_01x04, J11 Conn_01x04, J12 Conn_01x04, J13 Conn_01x02, J14 Conn_01x02, J15 Conn_01x02, J16 Conn_01x02, J17 Conn_01x02, J18 Conn_01x06, J19 Conn_01x06, J2 Conn_01x03, J20 Conn_01x06, J21 Conn_01x06, J22 Conn_01x02, J23 Conn_01x02, J24 Conn_01x02, J25 Conn_01x02, J26 Conn_01x06, J27 Conn_01x07, J28 Conn_01x03, J29 Conn_01x03, J3 Conn_01x04, J30 Conn_01x03, J31 Conn_01x03, J32 Conn_01x03, J33 Conn_01x03, J34 Conn_01x03, J35 Conn_01x03, J4 Conn_01x02, J5 Conn_01x06, J6 Conn_01x05, J7 Conn_01x03, J8 Conn_01x06, J9 Conn_01x04, U2 ADAU1452, U4 AMS1117-1.2, X1 12.288MHz

Commit message: Added Initial Firmware
Routing:
- net GND: track 196.3 -> 193.4 mm
Other:
- board text added: "V0.5"
- board text removed: "V0.4"
Changed lines of the file:
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@@
 		)
 	)
-	(gr_text "V0.4"
+	(gr_text "V0.5"
 		(at 120.9812 90.7876 0)
 		(layer "F.SilkS")
@@
 	)
 	(segment
-		(start 72.775248 91.08955)
-		(end 72.503748 91.08955)
-		(width 0.2)
-		(layer "F.Cu")
-		(net 2)
-	)
-	(segment
 		(start 85.8774 81.3816)
 		(end 86.6648 81.3816)
@@
 	)
 	(segment
-		(start 68.6054 89.8062)
-		(end 68.6054 89.5604)
-		(width 0.2)
-		(layer "F.Cu")
-		(net 2)
-	)
-	(segment
 		(start 94.1618 81.3562)
 		(end 94.9452 81.3562)
@@
 		(width 0.2)
 		(layer "F.Cu")
-		(net 2)
-	)
-	(segment
-		(start 66.8602 117.1209)
-		(end 68.6102 118.8709)
-		(width 0.2)
-		(layer "F.Cu")

Commit message: PCB V0.6 for second prototype
Parts:
- removed C1, C2, C5, C6, C8, C9: 10u, Capacitor_SMD:C_0603_1608Metric
- removed C12, C14, C16, C17, C18, C19: 100n, Capacitor_SMD:C_0402_1005Metric
- removed C33, C35, C36, C7: 2.2u, Capacitor_SMD:C_0402_1005Metric
- removed C60, C61, C62, C63, C64, C65, C66, C67, C68, C69, C70, C71, C72, C73, C74, C75, C76, C77, C78, C79, C80, C81, C82, C83, C84, C85, C86, C87, C88, C89, C90, C91: 1u, Capacitor_SMD:C_0402_1005Metric
- removed J1, J2, J28, J29, J30, J31, J32, J33, J34, J35, J7: Conn_01x03, Connector_PinHeader_2.54mm:PinHeader_1x03_P2.54mm_Vertical
- removed J10, J11, J12, J9: Conn_01x04, Connector_PinHeader_2.54mm:PinHeader_1x04_P2.54mm_Vertical
- removed J13, J4: Conn_01x02, Connector_PinHeader_2.54mm:PinHeader_1x02_P2.54mm_Vertical
- removed J20, J21, J26, J8: Conn_01x06, Connector_PinHeader_2.54mm:PinHeader_1x06_P2.54mm_Vertical
- removed J27: Conn_01x07, Connector_PinHeader_2.54mm:PinHeader_1x07_P2.54mm_Vertical
- removed J6: Conn_01x05, Connector_PinHeader_2.54mm:PinHeader_1x05_P2.54mm_Vertical
- removed R10, R11: 10k, Resistor_SMD:R_0402_1005Metric
- removed R100, R101, R102, R103, R104, R105, R106, R107, R108, R109, R110, R111, R112, R113, R114, R115, R44, R45, R46, R47, R48, R49, R50, R51, R52, R53, R54, R55, R56, R57, R58, R59, R60, R61, R62, R63, R64, R65, R66, R67, R68, R69, R70, R71, R72, R73, R74, R75, R84, R85, R86, R87, R88, R89, R90, R91, R92, R93, R94, R95, R96, R97, R98, R99: 100k, Resistor_SMD:R_0402_1005Metric
- removed R36, R37, R38, R39, R40, R41, R42, R43, R76, R77, R78, R79, R80, R81, R82, R83: 220k, Capacitor_SMD:C_0603_1608Metric
- removed R9: 1k, Resistor_SMD:R_0402_1005Metric
- removed TP16, TP17, TP18, TP19, TP20, TP21, TP22, TP23, TP24, TP25, TP26, TP27, TP28, TP29, TP30, TP31: TestPoint, TestPoint:TestPoint_THTPad_D2.0mm_Drill1.0mm
- removed U1, U5: ~, Custom:AK4619VN
- removed U10, U11, U12, U13: ~, Custom:LM324DT
Connections:
- net /EN renamed /uC_EN
Routing:
- net /MCLK: track 155.1 -> 0.00 mm, vias 3 -> 0
- net /AOUT4: track 92.1 -> 0.00 mm, vias 1 -> 0
- net /AOUT3: track 84.3 -> 0.00 mm, vias 1 -> 0
- net /AOUT2: track 84.0 -> 0.00 mm, vias 1 -> 0
- net /AOUT7: track 80.7 -> 0.00 mm, vias 1 -> 0
- net /AOUT6: track 80.3 -> 0.00 mm, vias 1 -> 0
- net /AOUT8: track 87.8 -> 10.2 mm, vias 1 -> 0
- net GND: track 193.4 -> 121.0 mm, vias 109 -> 57
- net /AOUT1: track 78.3 -> 7.75 mm, vias 1 -> 0
- net /LRCLK_OUT0: track 67.5 -> 0.00 mm, vias 4 -> 0
- net /AOUT5: track 73.6 -> 7.75 mm, vias 1 -> 0
- net /BCLK_OUT0: track 65.2 -> 0.00 mm, vias 4 -> 0
- net /BCLK_OUT1: track 53.6 -> 0.00 mm, vias 3 -> 0
- net +3V3: track 112.1 -> 63.7 mm, vias 33 -> 7
- net /SDATA_OUT0: track 44.4 -> 0.00 mm, vias 2 -> 0
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Other:
- board text removed: "Balanced Input"
