File: PCB/DIYDSPv0.5/DIYDSPv0.5.kicad_sch (KiCad schematic)
At the start: 292 parts, among them J1 Conn_01x03, J10 Conn_01x04, J11 Conn_01x04, J12 Conn_01x04, J13 Conn_01x02, J14 Conn_01x02, J15 Conn_01x02, J16 Conn_01x02, J17 Conn_01x02, J18 Conn_01x06, J19 Conn_01x06, J2 Conn_01x03, J20 Conn_01x06, J21 Conn_01x06, J22 Conn_01x02, J23 Conn_01x02, J24 Conn_01x02, J25 Conn_01x02, J26 Conn_01x06, J27 Conn_01x07, J28 Conn_01x03, J29 Conn_01x03, J3 Conn_01x04, J30 Conn_01x03, J31 Conn_01x03, J32 Conn_01x03, J33 Conn_01x03, J34 Conn_01x03, J35 Conn_01x03, J4 Conn_01x02, J5 Conn_01x06, J6 Conn_01x05, J7 Conn_01x03, J8 Conn_01x06, J9 Conn_01x04, U2 ADAU1452, U4 AMS1117-1.2, X1 12.288MHz

Commit message: PCB V0.6 for second prototype
Parts:
- removed C1, C2, C5, C52, C54, C55, C58, C59, C6, C8, C9: 10u, Capacitor_SMD:C_0603_1608Metric, symbol Device:C
- removed C12, C14, C16, C17, C18, C19: 100n, Capacitor_SMD:C_0402_1005Metric, symbol Device:C
- removed C33, C35, C36, C7: 2.2u, Capacitor_SMD:C_0402_1005Metric, symbol Device:C
- removed C64, C65, C72, C73, C74, C75, C80, C81, C82, C83, C88, C89, C90, C91: 1u, Capacitor_SMD:C_0402_1005Metric, symbol Device:C
- removed J1, J2, J28, J29, J30, J31, J32, J33, J34, J35, J7: Conn_01x03, Connector_PinHeader_2.54mm:PinHeader_1x03_P2.54mm_Vertical, symbol Connector_Generic:Conn_01x03
- removed J10, J11, J12, J9: Conn_01x04, Connector_PinHeader_2.54mm:PinHeader_1x04_P2.54mm_Vertical, symbol Connector_Generic:Conn_01x04
- removed J14, J15, J16, J17, J22, J23, J24, J25: Conn_01x02, Connector_PinHeader_2.54mm:PinHeader_1x02_P2.54mm_Vertical, symbol Connector_Generic:Conn_01x02
- removed J18, J19, J20, J21, J26: Conn_01x06, Connector_PinHeader_2.54mm:PinHeader_1x06_P2.54mm_Vertical, symbol Connector_Generic:Conn_01x06
- removed J27: Conn_01x07, Connector_PinHeader_2.54mm:PinHeader_1x07_P2.54mm_Vertical, symbol Connector_Generic:Conn_01x07
- removed R104, R105, R106, R107, R112, R113, R114, R115, R12, R13, R20, R22, R23, R26, R34, R48, R49, R56, R57, R66, R74, R88, R89, R96, R97, R98, R99: 100k, Resistor_SMD:R_0402_1005Metric, symbol Device:R
- removed R16, R17, R28, R30, R31, R40, R41, R80, R81: 220k, Capacitor_SMD:C_0603_1608Metric, symbol Device:R
- removed TP12, TP14, TP20, TP21, TP28, TP29, TP30, TP31, TP8, TP9: TestPoint, TestPoint:TestPoint_THTPad_D2.0mm_Drill1.0mm, symbol Connector:TestPoint
- removed U1, U5: ~, Custom:AK4619VN, symbol AK4619VN:AK4619VN
- removed U12, U13, U8: ~, Custom:LM324DT, symbol LM324DT:LM324DT
- added C40, C41, C44, C45, C47, C50, C51, C60, C61, C63, C69: 1u, Capacitor_SMD:C_0402_1005Metric, symbol Device:C
- added J2, J3: Conn_02x10_Odd_Even, Connector_PinHeader_2.54mm:PinHeader_2x10_P2.54mm_Vertical, symbol Connector_Generic:Conn_02x10_Odd_Even
- added R38, R39, R46, R47, R61, R69, R78, R79, R86, R87: 100k, Resistor_SMD:R_0402_1005Metric, symbol Device:R
- added R54, R55: 220k, Capacitor_SMD:C_0603_1608Metric, symbol Device:R
- added TP18, TP19: TestPoint, TestPoint:TestPoint_THTPad_D2.0mm_Drill1.0mm, symbol Connector:TestPoint
- added U9: ~, Custom:LM324DT, symbol LM324DT:LM324DT
- C53, C56, C57: value 10u -> 1u; footprint Capacitor_SMD:C_0603_1608Metric -> Capacitor_SMD:C_0402_1005Metric; LCSC Part # C96446 -> C52923
- R14, R15, R58, R59: value 100k -> 220k; footprint Resistor_SMD:R_0402_1005Metric -> Capacitor_SMD:C_0603_1608Metric; LCSC Part # C25741 -> C22961
- R29, R42, R43, R82, R83: value 220k -> 100k; footprint Capacitor_SMD:C_0603_1608Metric -> Resistor_SMD:R_0402_1005Metric; LCSC Part # C22961 -> C25741
- renumbered C92 to C1, C21 to C10, C22 to C11, C23 to C12, C24 to C13, C25 to C14, C26 to C15, C27 to C16, C28 to C17, C29 to C18, C30 to C19, C3 to C2, C31 to C20, C32 to C21, C34 to C22, C37 to C23, C38 to C24, C39 to C25, C40 to C26, C41 to C27, C42 to C28, C43 to C29, C4 to C3, C44 to C30, C45 to C31, C46 to C32, C47 to C33, C48 to C34, C49 to C35, C50 to C36, C51 to C37, C60 to C38, C61 to C39, C93 to C4, C62 to C42, C63 to C43, C68 to C46, C69 to C48, C70 to C49, C10 to C5, C71 to C52, C76 to C54, C77 to C55, C78 to C58, C79 to C59, C11 to C6, C84 to C62, C85 to C64, C86 to C65, C87 to C68, C13 to C7, C15 to C8, C20 to C9, J3 to J1, J8 to J7, J13 to J8, R36 to R12, R37 to R13, R38 to R16, R39 to R17, R44 to R20, R45 to R22, R46 to R23, R47 to R26, R52 to R28, R53 to R30, R54 to R31, R55 to R34, R60 to R36, R61 to R37, R62 to R40, R63 to R41, R68 to R44, R69 to R45, R70 to R48, R71 to R49, R76 to R52, R77 to R53, R78 to R56, R79 to R57, R84 to R60, R85 to R62, R86 to R63, R87 to R66, R92 to R68, R93 to R70, R94 to R71, R95 to R74, R100 to R76, R101 to R77, R102 to R80, R103 to R81, R108 to R84, R109 to R85, R110 to R88, R111 to R89, TP18 to TP12, TP19 to TP14, TP24 to TP16, TP25 to TP17, TP26 to TP20, TP27 to TP21, TP16 to TP8, TP17 to TP9, U2 to U1, U3 to U2, U4 to U3, U6 to U4, U9 to U5, U10 to U6, U11 to U8
Connections:
- net AIN2N is gone; now on net ADC_IN4: C64.2, R77.2, R85.2
- net AIN4N is gone; now on net ADC_IN8: C68.2, R81.2, R89.2
- net AIN4P is gone; now on net ADC_IN7: C65.2, R80.2, R88.2
- net +12V: now also R21.1, R24.1, R25.1, R27.1, R64.1, R65.1, R67.1, R61.1, U9.4 (VCC+); no longer R50.1, R51.1, R90.1, R91.1
- net +3V3: now also R50.1, R51.1, R90.1, R91.1, J2.1 (Pin_1), J3.1 (Pin_1), R46.1, R47.1, R86.1, R87.1; no longer R72.1, R73.1, R75.1
- net AOUT1: now also C47.2, J3.11 (Pin_11), R38.2, R46.2; no longer TP10.1
- net AOUT2: now also C50.2, J3.13 (Pin_13), R39.2, R47.2
- net AOUT3: now also J3.15 (Pin_15); no longer TP11.1
- net AOUT4: now also J3.17 (Pin_17); no longer TP15.1
- net AOUT5: now also R42.2, R50.2, C51.2, J3.12 (Pin_12); no longer U7.5 (IN2+)
- net AOUT6: now also C53.2, R43.2, R51.2, J3.14 (Pin_14); no longer U7.3 (IN1+)
- net AOUT7: now also J3.16 (Pin_16); no longer U7.10 (IN3+)
- net AOUT8: now also J3.18 (Pin_18); no longer TP13.1, U7.12 (IN4+)
- net BCLK_OUT0: now also J2.6 (Pin_6)
- net BCLK_OUT1: now also J2.10 (Pin_10)
- net BCLK_OUT2: now also J2.14 (Pin_14)
- net BCLK_OUT3: now also J2.18 (Pin_18)
- net EN: now also J2.20 (Pin_20); no longer U5.3 (EN)
- net GND: now also R29.1, R32.1, R33.1, R35.1, R42.1, R43.1, R72.1, R73.1, R75.1, R82.1, R83.1, J2.2 (Pin_2), J3.2 (Pin_2), R38.1, R39.1, R69.1, R78.1, R79.1, U9.11 (VCC-); no longer R14.2, R15.2, R21.2, R24.2, R25.2, R27.2, R32.2, R33.2, R35.2, R58.1, R59.1, R64.1, R65.1, R67.1
- net LRCLK_OUT0: now also J2.5 (Pin_5)
- net LRCLK_OUT1: now also J2.9 (Pin_9)
- net LRCLK_OUT2: now also J2.13 (Pin_13)
- net LRCLK_OUT3: now also J2.17 (Pin_17)
- net MCLK: now also J2.19 (Pin_19)
- net SCL: now also J3.20 (Pin_20)
- net SDA: now also J3.19 (Pin_19)
- net SDATA_IN0: now also J2.3 (Pin_3)
- net SDATA_IN1: now also J2.7 (Pin_7)
- net SDATA_IN2: now also J2.11 (Pin_11)
- net SDATA_IN3: now also J2.15 (Pin_15)
- net SDATA_OUT0: now also J2.4 (Pin_4)
- net SDATA_OUT1: now also J2.8 (Pin_8)
- net SDATA_OUT2: now also J2.12 (Pin_12)
- net SDATA_OUT3: now also J2.16 (Pin_16)
- net at TP22.1: now also C67.1, U9.8 (OUT3), U9.9 (IN3-)
- net AIN1: now reaches C38.1
- net AIN1: now also J3.3 (Pin_3)
- net AIN2: now reaches C39.1
- net AIN2: now also J3.5 (Pin_5)
- net AIN3: now reaches C54.1
- net AIN3: now also J3.7 (Pin_7)
- net at U7.1 (OUT1): now also TP10.1, U7.2 (IN1-), C47.1; no longer C56.1
- net at C57.2: now also R55.1; no longer R33.1
- net at U7.9 (IN3-): now also U7.8 (OUT3), C63.1, TP18.1
- net AIN8: now reaches C59.1
- net AIN8: now also C61.1, J3.10 (Pin_10)
- net at TP23.1: now also C69.1, U9.13 (IN4-), U9.14 (OUT4)
- net at R19.1: now also C45.2
- net AIN5: now reaches C42.1
- net AIN5: now also J3.4 (Pin_4)
- net AIN6: now reaches C43.1
- net AIN6: now also J3.6 (Pin_6)
- net at U7.6 (IN2-): now also TP11.1, U7.7 (OUT2), C50.1
- net at R18.2: now also R25.2, R33.2, U9.3 (IN1+); no longer R14.1
- net at R18.1: now also C44.2
- net at C53.1: now also TP15.1, U9.6 (IN2-), U9.7 (OUT2); no longer U7.8 (OUT3)
- net ADC_IN8: now reaches R83.2, R91.2
- net ADC_IN8: now also C69.2
- net AIN7: now reaches C58.1
- net AIN7: now also C60.1, J3.8 (Pin_8)
- net at C66.1: now also U7.13 (IN4-), U7.14 (OUT4), TP19.1
- net AIN4: now reaches C55.1
- net AIN4: now also J3.9 (Pin_9)
- net ADC_IN7: now reaches R82.2, R90.2
- net ADC_IN7: now also C67.2
- net ADC_IN4: now reaches C66.2
- net ADC_IN4: now also R79.2, R87.2; no longer R42.1
- net at C56.2: now also R54.1; no longer R32.1
- net at R19.2: now also R27.2, R35.2, U9.5 (IN2+); no longer R15.1
- net AIN1N renamed ADC_IN2
- net AIN1P renamed ADC_IN1
- net AIN2P renamed ADC_IN3
- net ADC_IN3: now also C63.2, R78.2, R86.2
- net AIN3N renamed ADC_IN6
- net AIN3P renamed ADC_IN5
- net AIN5N: no longer names the net of R65.2, R73.2
- net AIN5N: now also R58.2, U9.10 (IN3+)
- net AIN5P: no longer names the net of R64.2, R72.2
- net AIN5P: now also U7.12 (IN4+), R55.2
- net AIN7N: no longer names the net of R67.2, R75.2
- net AIN7N: now also R59.2, U9.12 (IN4+)
- new net: C60.2, R58.1
- new net: R54.2, R61.2, R69.2, U7.10 (IN3+)
- new net: R15.2, R24.2, R32.2, U7.5 (IN2+)
- new net: R14.2, R21.2, R29.2, U7.3 (IN1+)
- new net: C41.2, R15.1
- new net: C61.2, R59.1
- new net: C40.2, R14.1
- new net: C51.1, TP13.1, U9.1 (OUT1), U9.2 (IN1-)
- new net DAC_OUT1: C40.1
- new net DAC_OUT2: C41.1
- new net DAC_OUT3: C56.1
- new net DAC_OUT4: C57.1
- new net DAC_OUT5: C44.1
- new net DAC_OUT6: C45.1
- new net uC_EN: U5.3 (EN)
Other:
- note added: "12-16V DC IN"
- note added: "Analog Output"
- note added: "CODEC Connectors"
- note removed: "10-20V IN"
- note removed: "AK4619"
- note removed: "AK4619 Power Nets & Connectors"
- note removed: "Analog Out"
- note removed: "ESP32 Breakout"
- moved on the sheet: U5
