File: PCB/DIYDSPv0.8/DIYDSPv0.8.kicad_pcb (KiCad board)
At the start: 4 copper layers, 100 x 65 mm, 260 parts, among them J1 Conn_01x06, J10 Conn_01x05, J11 Conn_01x05, J12 Conn_01x05, J13 Conn_01x05, J2 Conn_01x05, J3 Conn_01x04, J4 Conn_01x04, J5 Conn_01x02, J6 Conn_01x05, J7 Conn_01x05, J8 Conn_01x05, J9 Conn_01x05, U1 ADAU1452, U4 AMS1117-1.2, X1 12.288MHz

Commit message: Added DC polarity indicator to main board, created RCA and XLR input/output
Other:
- board text added: "+ -"
- board text added: "12V DC"
Changed lines of the file:
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@@
+		)
+	)
+	(gr_text "12V DC"
+		(at 34.8 45.95 0)
+		(layer "B.SilkS")
+		(effects
+			(font
+				(size 1.6 1.6)
+				(thickness 0.32)
+				(bold yes)
+			)
+			(justify left bottom mirror)
 		)
 	)
@@
 		)
 	)
+	(gr_text "+\n\n-"
+		(at 30.45 34.45 180)
+		(layer "B.SilkS")
+		(effects
+			(font
+				(size 1.6 1.6)
+				(thickness 0.32)
+				(bold yes)
+			)
+			(justify left bottom mirror)
+		)
+	)
