File: PCB/DIYDSPv0.8/DIYDSPv0.8.kicad_sch (KiCad schematic)
At the start: 199 parts, among them J1 Conn_01x06, J2 Conn_01x04, J3 Conn_01x04, J4 Conn_01x05, J5 Conn_01x01, J6 Conn_01x02, U1 ADAU1452, U5 AMS1117-1.2, X1 12.288MHz

Commit message: Backing up progress (starting bluetooth, DSP project not in linear state).
Connections:
- net +3V3: now also C53.2, U6.4 (VCC)
Changed lines of the file:
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@@
 	)
 	(junction
+		(at 176.53 170.18)
+		(diameter 0)
+		(color 0 0 0 0)
+	)
+	(junction
 		(at 130.81 53.34)
 		(diameter 0)
@@
 					(unit 1)
 				)
+			)
+		)
+	)
+	(symbol
+		(lib_id "power:+3V3")
+		(at 176.53 170.18 0)
+		(unit 1)
+		(exclude_from_sim no)
+		(in_bom yes)
+		(on_board yes)
+		(dnp no)
+		(fields_autoplaced yes)
+		(property "Reference" "#PWR0146"
+			(at 176.53 173.99 0)
+			(effects
+				(font
+					(size 1.27 1.27)
+				)
+				(hide yes)
+			)
+		)
+		(property "Value" "+3V3"
+			(at 176.53 165.1 0)
+			(effects
+				(font
+					(size 1.27 1.27)
+				)
+			)
+		)
+		(property "Footprint" ""
+			(at 176.53 170.18 0)
+			(effects
+				(font
+					(size 1.27 1.27)
+				)
+				(hide yes)
+			)
+		)
+		(property "Datasheet" ""
+			(at 176.53 170.18 0)
+			(effects
+				(font
+					(size 1.27 1.27)
+				)
+				(hide yes)
+			)
+		)
+		(property "Description" "Power symbol creates a global label with name \"+3V3\""
+			(at 176.53 170.18 0)
+			(effects
+				(font
+					(size 1.27 1.27)
+				)
+				(hide yes)
+			)
+		)
+		(pin "1"
+		)
+		(instances
+			(project ""
+				(path "/b7ce3e82-c245-4515-bd69-0cf398c79f59"
+					(reference "#PWR0146")
+					(unit 1)
+				)

Commit message: Updating progress on v0.8 design
Parts:
- removed C58, C59, C60, C61, C62, C63, C64, C65, C66, C67, C68, C69, C70, C71, C72, C73, C74, C75, C76, C77, C78, C79, C80, C81: 1u, Capacitor_SMD:C_0402_1005Metric, symbol Device:C
- removed J5: Conn_01x01, Connector_PinHeader_2.54mm:PinHeader_1x01_P2.54mm_Vertical, symbol Connector_Generic:Conn_01x01
- removed R25: 10k, Resistor_SMD:R_0402_1005Metric, symbol Device:R
- removed R29, R30, R37, R38, R39, R40, R41, R42, R43, R44, R45, R46, R49, R50, R57, R58, R59, R60, R61, R62, R63, R64, R65, R66: 100k, Resistor_SMD:R_0402_1005Metric, symbol Device:R
- removed R31, R32, R33, R34, R35, R36, R47, R48, R51, R52, R53, R54, R55, R56, R67, R68: 220k, Resistor_SMD:R_0603_1608Metric, symbol Device:R
- removed TP10, TP11, TP12, TP13, TP14, TP15, TP8, TP9: TestPoint, TestPoint:TestPoint_THTPad_D2.0mm_Drill1.0mm, symbol Connector:TestPoint
- removed U20, U21, U22, U23: ~, Custom:LM324DT, symbol LM324DT:LM324DT
- removed U4: ~, Custom:K7803M-1000R3, symbol K7803M-1000R3:K7803M-1000R3_C22749779
- added U4: ~, K7803-1000:PWRM-TH_K7803-1000, symbol Custom_Symbol:K7803-1000_C329334
Connections:
- net +12V: now also U4.1 (VIN)
- net +3V3: now also U4.3 (VOUT)
- net GND: now also U4.2 (GND)
Other:
- note added: "Digital Rail"
- note removed: "3.3V Source"
- note removed: "Analog Input"
- note removed: "Analog Out"

Commit message: v0.8 hardware schematic mostly complete
Parts:
- removed C10, C11, C12: 22u, Capacitor_SMD:C_0805_2012Metric, symbol Device:C
- removed C48: 100n, Capacitor_SMD:C_0402_1005Metric, symbol Device:C
- removed R14: 100k, Resistor_SMD:R_0402_1005Metric, symbol Device:R
- removed TP1, TP3: TestPoint, TestPoint:TestPoint_THTPad_D4.0mm_Drill2.0mm, symbol Connector:TestPoint
- removed U11, U12, U13, U14, U15, U16, U8, U9: ~, Custom:PJ-320D, symbol Custom_Symbol:PJ-320D_C22459515
- removed U18, U19, U7: ~, Custom:YTS1C0033BBG01, symbol Custom_Symbol:YTS1C0033BBG01
- added C100, C68, C83: 220uF, RVT1V221M0810:CAP-SMD_BD8.0-L8.3-W8.3-LS9.1-FD, symbol Custom_Symbol:RVT1V221M0810_C18221522
- added C101, C102, C107, C108, C111, C112, C58, C59, C64, C65, C76, C77, C84, C85, C96, C97: 10u, symbol Device:C
- added C103, C104, C113, C114, C51, C60, C61, C62, C66, C67, C73, C74, C75, C86, C87, C88, C89, C94, C98, C99: 100n, Capacitor_SMD:C_0402_1005Metric, symbol Device:C
- added C105, C106, C109, C110, C78, C95: 22u, Capacitor_SMD:C_0805_2012Metric, symbol Device:C
- added C54, C55, C56, C57, C69, C70, C71, C72, C79, C80, C81, C82, C90, C91, C92, C93: 1u, symbol Device:C
- added D4, D5: ~, CUS08F30,H3F:SOD-323F_L1.7-W1.3-LS2.5-RD, symbol Custom_Symbol:CUS08F30,H3F
- added H1, H2, H3, H4: MountingHole_Pad, symbol Mechanical:MountingHole_Pad
- added J10, J11, J12, J13, J6, J7, J8, J9: Conn_01x05, symbol Connector_Generic:Conn_01x05
- added R22: 100k, Resistor_SMD:R_0402_1005Metric, symbol Device:R
- added R28, R29, R44, R45, R56, R57, R70, R71: 1k, symbol Device:R
- added R30, R31, R32, R33, R34, R35, R36, R37, R38, R39, R40, R41, R42, R43, R46, R47, R48, R49, R50, R51, R52, R53, R54, R55, R58, R59, R60, R61, R62, R63, R64, R65, R66, R67, R68, R69, R72, R73, R74, R75, R76, R77, R78, R79: 100k, symbol Device:R
- added SW1, SW2, SW3: ~, Custom:TS110916043, symbol Custom_Symbol:TS110916043
- added TP4: TestPoint, TestPoint:TestPoint_THTPad_D2.0mm_Drill1.0mm, symbol Connector:TestPoint
- added U10, U11, U12, U13, U14, U15, U16, U17, U18, U19, U20, U21, U22, U24, U25, U8, U9: ~, TLV9062IDR:SOIC-8_L5.0-W4.0-P1.27-LS6.0-BL, symbol Custom_Symbol:TLV9062IDR
- added U26: ~, K7803-1000:PWRM-TH_K7803-1000, symbol Custom_Symbol:K7803-1000_C329334
- TP6: footprint TestPoint:TestPoint_THTPad_D4.0mm_Drill2.0mm -> TestPoint:TestPoint_THTPad_D2.0mm_Drill1.0mm
- renumbered C16 to C10, C17 to C11, C18 to C12, C19 to C13, C20 to C14, C21 to C15, C22 to C16, C23 to C17, C24 to C18, C13 to C19, C25 to C20, C27 to C21, C28 to C22, C29 to C23, C30 to C24, C31 to C25, C32 to C26, C33 to C27, C14 to C28, C35 to C29, C36 to C30, C37 to C31, C38 to C32, C39 to C33, C40 to C34, C41 to C35, C42 to C36, C26 to C37, C43 to C38, C44 to C39, C45 to C40, C46 to C41, C47 to C42, C34 to C43, C49 to C44, C50 to C45, C51 to C46, C52 to C47, C54 to C48, C56 to C49, C55 to C50, C57 to C52, C7 to C63, C8 to C7, C9 to C8, C15 to C9, D3 to D1, D4 to D2, D2 to D3, D1 to D6, J4 to J2, J2 to J3, J3 to J4, J6 to J5, R18 to R14, R19 to R17, R20 to R18, R23 to R19, R24 to R20, R26 to R21, R21 to R23, R22 to R24, R17 to R25, R27 to R26, R28 to R27, TP4 to TP1, TP7 to TP2, TP2 to TP3, U4 to U23, U5 to U4, U17 to U5, U10 to U7
Connections:
- net +12V: now also C60.2, D5.2 (A); no longer C63.2, D6.2, TP3.1, U23.1 (VIN)
- net +3V3: now also C106.1; no longer C11.2, C12.2, C13.2, C18.1, C20.1, C21.2, C24.2, C27.2, R21.1, U2.18 (AVDD), U2.21 (VREFH), U3.18 (AVDD), U3.21 (VREFH)
- net BCLK_OUT0: now also R3.1; no longer R6.1
- net BCLK_OUT1: now also R6.1; no longer R3.1
- net DAC_OUT1: now also R28.2
- net DAC_OUT2: now also R44.2
- net DAC_OUT3: now also R56.2
- net DAC_OUT4: now also R70.2
- net DAC_OUT5: now also R29.2
- net DAC_OUT6: now also R45.2
- net DAC_OUT7: now also R57.2
- net DAC_OUT8: now also R71.2
- net EN: now also SW1.3
- net GND: now also C100.2, C103.2, C104.2, C105.2, C106.2, C109.2, C110.2, C113.2, C114.2, C51.1, C60.1, C61.2, C62.2, C66.2, C67.2, C68.2, C73.2, C74.2, C75.1, C78.1, C83.2, C86.2, C87.2, C88.2, C89.2, C94.1, C95.1, C98.2, C99.2, H1.1, H2.1, H3.1, H4.1, J10.1 (Pin_1), J11.1 (Pin_1), J12.1 (Pin_1), J13.1 (Pin_1), J6.1 (Pin_1), J7.1 (Pin_1), J8.1 (Pin_1), J9.1 (Pin_1), R22.1, R69.2, R75.2, SW1.4, SW2.1, SW3.1, U10.4 (VEE/GND), U11.4 (VEE/GND), U12.4 (VEE/GND), U13.4 (VEE/GND), U14.4 (VEE/GND), U15.4 (VEE/GND), U16.4 (VEE/GND), U17.4 (VEE/GND), U18.4 (VEE/GND), U19.4 (VEE/GND), U20.4 (VEE/GND), U21.4 (VEE/GND), U22.4 (VEE/GND), U24.4 (VEE/GND), U25.4 (VEE/GND), U26.2 (GND), U8.4 (VEE/GND), U9.4 (VEE/GND); no longer TP6.1
- net IO0: now also SW2.2
- net LRCLK_OUT0: now also R2.1; no longer R5.1
- net LRCLK_OUT1: now also R5.1; no longer R2.1
- net SDATA_IN0: now also R10.1; no longer R11.1
- net SDATA_IN1: now also R11.1; no longer R10.1
- net SDATA_OUT0: now also R8.1; no longer R9.1
- net SDATA_OUT1: now also R9.1; no longer R8.1
- net at U6.3 (MR#): now also C51.2, SW3.2
- net VBUS: now reaches U7.A4B9 (VBUS)
- net VBUS: now also U7.B4A9 (VBUS), C75.2, D4.2 (A)
- net ADC_IN7N: now reaches U3.11 (IN3N/AIN5L/GND6L)
- net ADC_IN7N: now also U17.6 (INB-), U17.7 (OUTB)
- net ADC_IN6N: now reaches U3.13 (IN2N/AIN2R/GND3R)
- net ADC_IN6N: now also U13.6 (INB-), U13.7 (OUTB)
- net ADC_IN5N: now reaches U3.15 (IN1N/AIN2L/GND3L)
- net ADC_IN5N: now also U9.6 (INB-), U9.7 (OUTB)
- net ADC_IN8N: now reaches U3.9 (IN4N/AIN5R/GND6R)
- net ADC_IN8N: now also U19.6 (INB-), U19.7 (OUTB)
- net ADC_IN3N: now reaches U2.11 (IN3N/AIN5L/GND6L)
- net ADC_IN3N: now also U16.6 (INB-), U16.7 (OUTB)
- net ADC_IN2N: now reaches U2.13 (IN2N/AIN2R/GND3R)
- net ADC_IN2N: now also U12.6 (INB-), U12.7 (OUTB)
- net ADC_IN1N: now reaches U2.15 (IN1N/AIN2L/GND3L)
- net ADC_IN1N: now also U8.6 (INB-), U8.7 (OUTB)
- net ADC_IN4N: now reaches U2.9 (IN4N/AIN5R/GND6R)
- net ADC_IN4N: now also U18.6 (INB-), U18.7 (OUTB)
- net ADC_IN1 renamed ADC_IN1P
- net ADC_IN1P: now also U10.1 (OUTA), U10.2 (INA-)
- net ADC_IN2 renamed ADC_IN2P
- net ADC_IN2P: now also U12.1 (OUTA), U12.2 (INA-)
- net ADC_IN3 renamed ADC_IN3P
- net ADC_IN3P: now also U16.1 (OUTA), U16.2 (INA-)
- net ADC_IN4 renamed ADC_IN4P
- net ADC_IN4P: now also U20.1 (OUTA), U20.2 (INA-)
- net ADC_IN5 renamed ADC_IN5P
- net ADC_IN5P: now also U11.1 (OUTA), U11.2 (INA-)
- net ADC_IN6 renamed ADC_IN6P
- net ADC_IN6P: now also U13.1 (OUTA), U13.2 (INA-)
- net ADC_IN7 renamed ADC_IN7P
- net ADC_IN7P: now also U17.1 (OUTA), U17.2 (INA-)
- net ADC_IN8 renamed ADC_IN8P
- net ADC_IN8P: now also U21.1 (OUTA), U21.2 (INA-)
- removed net CODEC_PDN: U2.26 (PDN), U3.26 (PDN), U6.2 (RESET#/RESET)
- new net: R29.1, R31.1, U9.3 (INA+)
- new net: C92.1, R62.1, U21.3 (INA+)
- new net: C90.1, R60.1, U20.3 (INA+)
- new net: C101.2, R66.1, U20.7 (OUTB)
- new net: R64.1, R66.2, U20.6 (INB-)
- new net: C80.1, R51.2, U16.5 (INB+)
- new net: R70.1, R72.1, U24.3 (INA+)
- new net: C82.1, R53.2, U17.5 (INB+)
- new net: C70.1, R41.2, U12.5 (INB+)
- new net: C65.2, R39.1, U11.7 (OUTB)
- new net: C55.1, R33.2, U8.5 (INB+)
- new net: R56.1, R58.1, U18.3 (INA+)
- new net: R49.1, R55.2, U15.6 (INB-)
- new net: C77.2, R49.2, U15.1 (OUTA), U15.2 (INA-)
- new net: C108.2, R77.2, U25.1 (OUTA), U25.2 (INA-)
- new net: R71.1, R73.1, U25.3 (INA+)
- new net: C76.2, R48.2, U14.1 (OUTA), U14.2 (INA-)
- new net: R44.1, R46.1, U14.3 (INA+)
- new net: R57.1, R59.1, U19.3 (INA+)
- new net: R28.1, R30.1, U8.3 (INA+)
- new net: C79.1, R50.1, U16.3 (INA+)
- new net: C85.2, R55.1, U15.7 (OUTB)
- new net: C57.1, R35.2, U9.5 (INB+)
- new net: R65.1, R67.2, U21.6 (INB-)
- new net: C97.2, R65.2, U19.1 (OUTA), U19.2 (INA-)
- new net: C54.1, R32.1, U10.3 (INA+)
- new net: R74.2, R75.1, U22.5 (INB+)
- new net: R76.1, R78.2, U24.6 (INB-)
- new net: C111.2, R78.1, U24.7 (OUTB)
- new net: C59.2, R37.2, U9.1 (OUTA), U9.2 (INA-)
- new net: C107.2, R76.2, U24.1 (OUTA), U24.2 (INA-)
- new net: C56.1, R34.1, U11.3 (INA+)
- new net: C91.1, R61.2, U18.5 (INB+)
- new net: C96.2, R64.2, U18.1 (OUTA), U18.2 (INA-)
- new net: C63.2, C68.1, TP3.1
- new net: C112.2, R79.1, U25.7 (OUTB)
- new net: R77.1, R79.2, U25.6 (INB-)
- new net: R68.2, R69.1, U22.3 (INA+)
- new net: R36.1, R38.2, U10.6 (INB-)
- new net: C58.2, R36.2, U8.1 (OUTA), U8.2 (INA-)
- new net: C78.2, C83.1, TP4.1
- new net: R48.1, R54.2, U14.6 (INB-)
- new net: C84.2, R54.1, U14.7 (OUTB)
- new net: C81.1, R52.1, U17.3 (INA+)
- new net: C71.1, R42.1, U13.3 (INA+)
- new net: C102.2, R67.1, U21.7 (OUTB)
- new net: C72.1, R43.2, U13.5 (INB+)
- new net: R21.1, R22.2, U6.2 (RESET#/RESET)
- new net: C69.1, R40.1, U12.3 (INA+)
- new net: C93.1, R63.2, U19.5 (INB+)
- new net: R37.1, R39.2, U11.6 (INB-)
- new net: C64.2, R38.1, U10.7 (OUTB)
- new net: R45.1, R47.1, U15.3 (INA+)
- new net +3.3VA: C103.1, C104.1, C11.2, C110.1, C113.1, C114.1, C12.2, C13.2, C18.1, C20.1, C21.2, C24.2, C27.2, C61.1, C62.1, C66.1, C67.1, C73.1, C74.1, C86.1, C87.1, C88.1, C89.1, C98.1, C99.1, R68.1, R74.1, TP6.1, U10.8 (VCC), U11.8 (VCC), U12.8 (VCC), U13.8 (VCC), U14.8 (VCC), U15.8 (VCC), U16.8 (VCC), U17.8 (VCC), U18.8 (VCC), U19.8 (VCC), U2.18 (AVDD), U2.21 (VREFH), U20.8 (VCC), U21.8 (VCC), U22.8 (VCC), U24.8 (VCC), U25.8 (VCC), U26.3 (VOUT), U3.18 (AVDD), U3.21 (VREFH), U8.8 (VCC), U9.8 (VCC)
- new net 1V65_1: R32.2, R33.1, R34.2, R35.1, R40.2, R41.1, R42.2, R43.1, R50.2, R51.1, R52.2, R53.1, R60.2, R61.1, R62.2, R63.1, U22.1 (OUTA), U22.2 (INA-)
- new net 1V65_2: R30.2, R31.2, R46.2, R47.2, R58.2, R59.2, R72.2, R73.2, U10.5 (INB+), U11.5 (INB+), U14.5 (INB+), U15.5 (INB+), U20.5 (INB+), U21.5 (INB+), U22.6 (INB-), U22.7 (OUTB), U24.5 (INB+), U25.5 (INB+)
- new net AIN2_P: C69.2, J6.5 (Pin_5)
- new net AIN_1N: C55.2, J6.2 (Pin_2)
- new net AIN_1P: C54.2, J6.3 (Pin_3)
- new net AIN_2N: C70.2, J6.4 (Pin_4)
- new net AIN_3N: C80.2, J8.2 (Pin_2)
- new net AIN_3P: C79.2, J8.3 (Pin_3)
- new net AIN_4N: C91.2, J8.4 (Pin_4)
- new net AIN_4P: C90.2, J8.5 (Pin_5)
- new net AIN_5N: C57.2, J10.2 (Pin_2)
- new net AIN_5P: C56.2, J10.3 (Pin_3)
- new net AIN_6N: C72.2, J10.4 (Pin_4)
- new net AIN_6P: C71.2, J10.5 (Pin_5)
- new net AIN_7N: C82.2, J12.2 (Pin_2)
- new net AIN_7P: C81.2, J12.3 (Pin_3)
- new net AIN_8N: C93.2, J12.4 (Pin_4)
- new net AIN_8P: C92.2, J12.5 (Pin_5)
- new net AOUT_1N: C64.1, J7.2 (Pin_2)
- new net AOUT_1P: C58.1, J7.3 (Pin_3)
- new net AOUT_2N: C84.1, J7.4 (Pin_4)
- new net AOUT_2P: C76.1, J7.5 (Pin_5)
- new net AOUT_3N: C101.1, J9.2 (Pin_2)
- new net AOUT_3P: C96.1, J9.3 (Pin_3)
- new net AOUT_4N: C111.1, J9.4 (Pin_4)
- new net AOUT_4P: C107.1, J9.5 (Pin_5)
- new net AOUT_5N: C65.1, J11.2 (Pin_2)
- new net AOUT_5P: C59.1, J11.3 (Pin_3)
- new net AOUT_6N: C85.1, J11.4 (Pin_4)
- new net AOUT_6P: C77.1, J11.5 (Pin_5)
- new net AOUT_7N: C102.1, J13.2 (Pin_2)
- new net AOUT_7P: C97.1, J13.3 (Pin_3)
- new net AOUT_8N: C112.1, J13.4 (Pin_4)
- new net AOUT_8P: C108.1, J13.5 (Pin_5)
- new net VCC: C100.1, C105.1, C109.1, C94.2, C95.2, D4.1 (C), D5.1 (C), D6.2, U23.1 (VIN), U26.1 (VIN)
- no-connect marks 73 -> 55
Other:
- note added: "Analog Output"
- note added: "Analog Rail"
- note added: "Analog input"
- note added: "ESP32"
- note added: "Power Input"
- note removed: "12V DC IN"
- note removed: "ADAU1452 AUXADC/MP"
- note removed: "ADAU1452 Clock Circuit"
- note removed: "ADAU1452 Power Nets"
- note removed: "AUX ESP32 Connections"
- note removed: "Audio Connectors"
- note removed: "ESP32 & Local Control"
- note removed: "Heartbeats"
- note removed: "PDN Generator"
- moved on the sheet: C1, C10, C11, C12, C13, C18, C19, C2, C20, C21, C24, C27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

Commit message: More progress on V0.8 layout. Still trying to figure out analog placement.
Parts:
- added C107: 220uF, Custom:RVT1V221M0810, symbol Custom_Symbol:RVT1V221M0810_C18221522
- added C116: 100n, Capacitor_SMD:C_0402_1005Metric, symbol Device:C
- added D3: ~, Custom:CUS08F30,H3F, symbol Custom_Symbol:CUS08F30,H3F
- added D8: LED, LED_SMD:LED_0805_2012Metric, symbol Device:LED
- added R15: 1k, Resistor_SMD:R_0402_1005Metric, symbol Device:R
- added R81: 100, Resistor_SMD:R_0805_2012Metric, symbol Device:R
- added TP5: TestPoint, TestPoint:TestPoint_THTPad_D2.0mm_Drill1.0mm, symbol Connector:TestPoint
- C100, C68, C83: footprint RVT1V221M0810:CAP-SMD_BD8.0-L8.3-W8.3-LS9.1-FD -> Custom:RVT1V221M0810; LCSC Part # (none) -> C18221522
- C101, C102, C58, C59, C64, C65, C76, C77, C84, C85, C96, C97: footprint (none) -> Capacitor_SMD:C_0603_1608Metric; LCSC Part # (none) -> C96446
- C108: renamed from C107; footprint (none) -> Capacitor_SMD:C_0603_1608Metric; LCSC Part # (none) -> C96446
- C109: renamed from C108; footprint (none) -> Capacitor_SMD:C_0603_1608Metric; LCSC Part # (none) -> C96446
- C112: renamed from C111; footprint (none) -> Capacitor_SMD:C_0603_1608Metric; LCSC Part # (none) -> C96446
- C113: renamed from C112; footprint (none) -> Capacitor_SMD:C_0603_1608Metric; LCSC Part # (none) -> C96446
- C54, C55, C56, C57, C69, C70, C71, C72, C79, C80, C81, C82, C90, C91, C92, C93: footprint (none) -> Capacitor_SMD:C_0402_1005Metric; LCSC Part # (none) -> C52923
- D4, D5: footprint CUS08F30,H3F:SOD-323F_L1.7-W1.3-LS2.5-RD -> Custom:CUS08F30,H3F; LCSC Part # (none) -> C150183
- H1, H2, H3, H4: footprint (none) -> MountingHole:MountingHole_3.2mm_M3_Pad_TopBottom
- J10, J11, J12, J13, J6, J7, J8, J9: footprint (none) -> Connector_PinHeader_2.54mm:PinHeader_1x05_P2.54mm_Vertical
- R28, R29, R44, R45, R56, R57, R70, R71: footprint (none) -> Resistor_SMD:R_0402_1005Metric; LCSC Part # (none) -> C11702
- R30, R31, R32, R33, R34, R35, R36, R37, R38, R39, R40, R41, R42, R43, R46, R47, R48, R49, R50, R51, R52, R53, R54, R55, R58, R59, R60, R61, R62, R63, R64, R65, R66, R67, R68, R69, R72, R73: footprint (none) -> Resistor_SMD:R_0402_1005Metric; LCSC Part # (none) -> C25741
- R75: renamed from R74; footprint (none) -> Resistor_SMD:R_0402_1005Metric; LCSC Part # (none) -> C25741
- R76: renamed from R75; footprint (none) -> Resistor_SMD:R_0402_1005Metric; LCSC Part # (none) -> C25741
- R77: renamed from R76; footprint (none) -> Resistor_SMD:R_0402_1005Metric; LCSC Part # (none) -> C25741
- R78: renamed from R77; footprint (none) -> Resistor_SMD:R_0402_1005Metric; LCSC Part # (none) -> C25741
- R79: renamed from R78; footprint (none) -> Resistor_SMD:R_0402_1005Metric; LCSC Part # (none) -> C25741
- R80: renamed from R79; footprint (none) -> Resistor_SMD:R_0402_1005Metric; LCSC Part # (none) -> C25741
- U10: renamed from U8; footprint TLV9062IDR:SOIC-8_L5.0-W4.0-P1.27-LS6.0-BL -> Custom:TLV9062IDR; LCSC Part # (none) -> C398355
- U10, U11, U12, U13, U14, U15, U16, U17, U18, U19, U20, U21, U22, U24, U25, U8, U9: footprint TLV9062IDR:SOIC-8_L5.0-W4.0-P1.27-LS6.0-BL -> Custom:TLV9062IDR; LCSC Part # (none) -> C398355
- U11: renamed from U9; footprint TLV9062IDR:SOIC-8_L5.0-W4.0-P1.27-LS6.0-BL -> Custom:TLV9062IDR; LCSC Part # (none) -> C398355
- U18: renamed from U20; footprint TLV9062IDR:SOIC-8_L5.0-W4.0-P1.27-LS6.0-BL -> Custom:TLV9062IDR; LCSC Part # (none) -> C398355
- U19: renamed from U21; footprint TLV9062IDR:SOIC-8_L5.0-W4.0-P1.27-LS6.0-BL -> Custom:TLV9062IDR; LCSC Part # (none) -> C398355
- U20: renamed from U18; footprint TLV9062IDR:SOIC-8_L5.0-W4.0-P1.27-LS6.0-BL -> Custom:TLV9062IDR; LCSC Part # (none) -> C398355
- U21: renamed from U19; footprint TLV9062IDR:SOIC-8_L5.0-W4.0-P1.27-LS6.0-BL -> Custom:TLV9062IDR; LCSC Part # (none) -> C398355
- U23, U26: footprint K7803-1000:PWRM-TH_K7803-1000 -> Custom:K7803-1000
- U8: renamed from U10; footprint TLV9062IDR:SOIC-8_L5.0-W4.0-P1.27-LS6.0-BL -> Custom:TLV9062IDR; LCSC Part # (none) -> C398355
- U9: renamed from U11; footprint TLV9062IDR:SOIC-8_L5.0-W4.0-P1.27-LS6.0-BL -> Custom:TLV9062IDR; LCSC Part # (none) -> C398355
- renumbered C105 to C103, C106 to C104, C103 to C105, C104 to C106, C109 to C110, C110 to C111, C113 to C114, C114 to C115, C38 to C36, C36 to C37, C37 to C38, C46 to C42, C42 to C43, C43 to C44, C44 to C45, C45 to C46, C63 to C61, C61 to C62, C62 to C63, D3 to D2, D2 to D7, R15 to R16, R16 to R17, R17 to R74, TP5 to TP6, TP6 to TP7
Connections:
- net +12V: now also C61.2, C68.1, TP3.1, D3.1 (C); no longer CN1.2
- net +3.3VA: now also C107.1, C116.1, R81.1
- net +3V3: now also R15.1
- net 1V65_1: now also U22.6 (INB-), U22.7 (OUTB); no longer U22.1 (OUTA), U22.2 (INA-)
- net 1V65_2: now also U22.1 (OUTA), U22.2 (INA-); no longer U22.6 (INB-), U22.7 (OUTB)
- net ADC_IN1N: now also U10.1 (OUTA), U10.2 (INA-); no longer U10.6 (INB-), U10.7 (OUTB)
- net ADC_IN1P: now also U10.6 (INB-), U10.7 (OUTB); no longer U10.1 (OUTA), U10.2 (INA-)
- net ADC_IN2N: now also U12.1 (OUTA), U12.2 (INA-); no longer U12.6 (INB-), U12.7 (OUTB)
- net ADC_IN2P: now also U12.6 (INB-), U12.7 (OUTB); no longer U12.1 (OUTA), U12.2 (INA-)
- net ADC_IN3N: now also U16.1 (OUTA), U16.2 (INA-); no longer U16.6 (INB-), U16.7 (OUTB)
- net ADC_IN3P: now also U16.6 (INB-), U16.7 (OUTB); no longer U16.1 (OUTA), U16.2 (INA-)
- net ADC_IN4N: now also U20.1 (OUTA), U20.2 (INA-); no longer U20.6 (INB-), U20.7 (OUTB)
- net ADC_IN4P: now also U20.6 (INB-), U20.7 (OUTB); no longer U20.1 (OUTA), U20.2 (INA-)
- net ADC_IN5N: now also U11.1 (OUTA), U11.2 (INA-); no longer U11.6 (INB-), U11.7 (OUTB)
- net ADC_IN5P: now also U11.6 (INB-), U11.7 (OUTB); no longer U11.1 (OUTA), U11.2 (INA-)
- net ADC_IN6N: now also U13.1 (OUTA), U13.2 (INA-); no longer U13.6 (INB-), U13.7 (OUTB)
- net ADC_IN6P: now also U13.6 (INB-), U13.7 (OUTB); no longer U13.1 (OUTA), U13.2 (INA-)
- net ADC_IN7N: now also U17.1 (OUTA), U17.2 (INA-); no longer U17.6 (INB-), U17.7 (OUTB)
- net ADC_IN7P: now also U17.6 (INB-), U17.7 (OUTB); no longer U17.1 (OUTA), U17.2 (INA-)
- net ADC_IN8N: now also U21.1 (OUTA), U21.2 (INA-); no longer U21.6 (INB-), U21.7 (OUTB)
- net ADC_IN8P: now also U21.6 (INB-), U21.7 (OUTB); no longer U21.1 (OUTA), U21.2 (INA-)
- net AIN2_P: now also C70.2, J6.4 (Pin_4); no longer C69.2, J6.5 (Pin_5)
- net AIN_1N: now also C54.2, J6.3 (Pin_3); no longer C55.2, J6.2 (Pin_2)
- net AIN_1P: now also C55.2, J6.2 (Pin_2); no longer C54.2, J6.3 (Pin_3)
- net AIN_2N: now also C69.2, J6.5 (Pin_5); no longer C70.2, J6.4 (Pin_4)
- net AIN_3N: now also C79.2, J8.3 (Pin_3); no longer C80.2, J8.2 (Pin_2)
- net AIN_3P: now also C80.2, J8.2 (Pin_2); no longer C79.2, J8.3 (Pin_3)
- net AIN_4N: now also C90.2, J8.5 (Pin_5); no longer C91.2, J8.4 (Pin_4)
- net AIN_4P: now also C91.2, J8.4 (Pin_4); no longer C90.2, J8.5 (Pin_5)
- net AIN_5N: now also C56.2, J10.3 (Pin_3); no longer C57.2, J10.2 (Pin_2)
- net AIN_5P: now also C57.2, J10.2 (Pin_2); no longer C56.2, J10.3 (Pin_3)
- net AIN_6N: now also C71.2, J10.5 (Pin_5); no longer C72.2, J10.4 (Pin_4)
- net AIN_6P: now also C72.2, J10.4 (Pin_4); no longer C71.2, J10.5 (Pin_5)
- net AIN_7N: now also C81.2, J12.3 (Pin_3); no longer C82.2, J12.2 (Pin_2)
- net AIN_7P: now also C82.2, J12.2 (Pin_2); no longer C81.2, J12.3 (Pin_3)
- net AIN_8N: now also C92.2, J12.5 (Pin_5); no longer C93.2, J12.4 (Pin_4)
- net AIN_8P: now also C93.2, J12.4 (Pin_4); no longer C92.2, J12.5 (Pin_5)
- net EN: now also R21.1; no longer R21.2
- net GND: now also C103.1, C51.2, R22.2, SW3.4, C107.2, C116.2, D8.1 (K); no longer C103.2, C51.1, R22.1, SW3.1
- net HB_LED1: now also R25.2; no longer R25.1
- net VBUS: now also C78.2, C83.1, TP4.1
- net VCC: now also C103.2, TP5.1; no longer C103.1
- net at D2.2 (A): now also R25.1; no longer R25.2
- net at SW3.3: now also C51.1, U6.3 (MR#)
- net CODEC_EN: now reaches U3.26 (PDN)
- net CODEC_EN: now also U2.26 (PDN), U5.22 (IO14), R15.2
- new net: CN1.2, D3.2 (A)
- new net: R21.2, R22.1, U6.2 (RESET#/RESET)
- new net: D8.2 (A), R81.2
- now unconnected: SW3.2
- no-connect marks 55 -> 54
Other:
- note added: "Pin15"
- note added: "Pin18"
- note added: "Pin2"
- note added: "Pin20"
- note added: "Pin35"
- note added: "Pin38"
- note added: "Pin53"
- note added: "Pin56"
- note added: "Pin7"
- note added: "Pin71"
- moved on the sheet: C103, C104, C36, C42, C51, D7, R21, R22, R25, R74, SW3, TP3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

Commit message: Nearly done with v0.8 placement - Dealing with DRC errors
Connections:
- net AOUT_1N: now also J7.3 (Pin_3); no longer J7.2 (Pin_2)
- net AOUT_1P: now also J7.2 (Pin_2); no longer J7.3 (Pin_3)
- net AOUT_2N: now also J7.5 (Pin_5); no longer J7.4 (Pin_4)
- net AOUT_2P: now also J7.4 (Pin_4); no longer J7.5 (Pin_5)
- net AOUT_3N: now also J9.3 (Pin_3); no longer J9.2 (Pin_2)
- net AOUT_3P: now also J9.2 (Pin_2); no longer J9.3 (Pin_3)
- net AOUT_4N: now also J9.5 (Pin_5); no longer J9.4 (Pin_4)
- net AOUT_4P: now also J9.4 (Pin_4); no longer J9.5 (Pin_5)
- net AOUT_5N: now also J11.3 (Pin_3); no longer J11.2 (Pin_2)
- net AOUT_5P: now also J11.2 (Pin_2); no longer J11.3 (Pin_3)
- net AOUT_6N: now also J11.5 (Pin_5); no longer J11.4 (Pin_4)
- net AOUT_6P: now also J11.4 (Pin_4); no longer J11.5 (Pin_5)
- net AOUT_7N: now also J13.3 (Pin_3); no longer J13.2 (Pin_2)
- net AOUT_7P: now also J13.2 (Pin_2); no longer J13.3 (Pin_3)
- net AOUT_8N: now also J13.5 (Pin_5); no longer J13.4 (Pin_4)
- net AOUT_8P: now also J13.4 (Pin_4); no longer J13.5 (Pin_5)
- net BCLK_OUT0: now also R6.1; no longer R3.1
- net BCLK_OUT1: now also R3.1; no longer R6.1
- net LRCLK_OUT0: now also R5.1; no longer R2.1
- net LRCLK_OUT1: now also R2.1; no longer R5.1
- net SDATA_IN0: now also R11.1; no longer R10.1
- net SDATA_IN1: now also R10.1; no longer R11.1
- net SDATA_OUT0: now also R9.1; no longer R8.1
- net SDATA_OUT1: now also R8.1; no longer R9.1
Changed lines of the file:
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@@
 	)
 	(label "AOUT_8P"
-		(at 565.15 148.59 0)
+		(at 565.15 151.13 0)
 		(effects
 			(font
@@
 	)
 	(label "AOUT_5N"
-		(at 544.83 156.21 0)
+		(at 544.83 153.67 0)
 		(effects
 			(font
@@
 	)
 	(label "AOUT_7P"
-		(at 565.15 153.67 0)
+		(at 565.15 156.21 0)
 		(effects
 			(font
@@
 		)
 	)
-	(label "BCLK_OUT0"
+	(label "BCLK_OUT1"
 		(at 40.64 219.71 180)
 		(effects
@@
 		)
 	)
-	(label "BCLK_OUT1"
+	(label "BCLK_OUT0"
 		(at 41.91 307.34 180)
 		(effects
@@
 		)
 	)
-	(label "SDATA_OUT1"
+	(label "SDATA_OUT0"
 		(at 45.72 292.1 180)
 		(effects
@@
 		)
 	)
-	(label "SDATA_OUT0"
+	(label "SDATA_OUT1"
 		(at 44.45 204.47 180)
 		(effects
@@
 	)
 	(label "AOUT_7N"
-		(at 565.15 156.21 0)
+		(at 565.15 153.67 0)
 		(effects
 			(font
@@
 	)
 	(label "AOUT_3P"
-		(at 524.51 153.67 0)
+		(at 524.51 156.21 0)
 		(effects
 			(font
@@
 	)
 	(label "AOUT_6P"
-		(at 544.83 148.59 0)
+		(at 544.83 151.13 0)
 		(effects
 			(font
@@
 		)
 	)
-	(label "LRCLK_OUT1"
+	(label "LRCLK_OUT0"
 		(at 41.91 304.8 180)
 		(effects
@@
 	)
 	(label "AOUT_1N"
-		(at 502.92 156.21 0)
+		(at 502.92 153.67 0)
 		(effects
 			(font
@@
 	)
 	(label "AOUT_3N"
-		(at 524.51 156.21 0)
+		(at 524.51 153.67 0)
 		(effects
 			(font
@@
 		)
 	)
-	(label "SDATA_IN0"
+	(label "SDATA_IN1"
 		(at 57.15 173.99 180)
 		(effects
@@
 	)
 	(label "AOUT_2N"
-		(at 502.92 151.13 0)
+		(at 502.92 148.59 0)
 		(effects
 			(font
@@
 		)
 	)
-	(label "LRCLK_OUT0"
+	(label "LRCLK_OUT1"
 		(at 40.64 217.17 180)
 		(effects
@@
 	)
 	(label "AOUT_5P"
-		(at 544.83 153.67 0)
+		(at 544.83 156.21 0)
 		(effects
 			(font
@@
 	)
 	(label "AOUT_4P"
-		(at 524.51 148.59 0)
+		(at 524.51 151.13 0)
 		(effects
 			(font
@@
 	)
 	(label "AOUT_6N"
-		(at 544.83 151.13 0)
+		(at 544.83 148.59 0)
 		(effects
 			(font
@@
 	)
 	(label "AOUT_4N"
-		(at 524.51 151.13 0)
+		(at 524.51 148.59 0)
 		(effects
 			(font
@@
 	)
 	(label "AOUT_8N"
-		(at 565.15 151.13 0)
-		(effects
-			(font
-				(size 1.27 1.27)
-			)
-			(justify left bottom)
-		)
-	)
-	(label "SDATA_IN1"
+		(at 565.15 148.59 0)
+		(effects
+			(font
+				(size 1.27 1.27)
+			)
+			(justify left bottom)
+		)
+	)
+	(label "SDATA_IN0"
 		(at 58.42 261.62 180)
 		(effects
@@
 	)
 	(label "AOUT_2P"
-		(at 502.92 148.59 0)
+		(at 502.92 151.13 0)
 		(effects
 			(font
@@
 	)
 	(label "AOUT_1P"
-		(at 502.92 153.67 0)
-		(effects
-			(font
+		(at 502.92 156.21 0)
+		(effects
+			(font

Commit message: V0.8 Complete. Will be working on audio connector boards.
Parts:
- removed U23, U26: ~, Custom:K7803-1000, symbol Custom_Symbol:K7803-1000_C329334
- added U23, U26: ~, Custom:K7803-1000_C50396471, symbol Custom_Symbol:K7803-1000_C50396471
- J1, J10, J11, J12, J13, J2, J3, J4, J5, J6, J7, J8, J9: now not fitted
Connections:
- net +3.3VA: now also U26.3 (VOUT)
- net +3V3: now also U23.3 (VOUT)
- net GND: now also U23.2 (GND), U26.2 (GND)
- net VCC: now also U23.1 (VIN), U26.1 (VIN)

Commit message: Updated v0.8 PCB for final version and added version for external ESP32 dev board.
Connections:
- net +3V3: no longer R15.1
- net GND: now also R15.1
Changed lines of the file:
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@@
 	)
 	(symbol
-		(lib_id "power:+3V3")
-		(at 125.73 184.15 180)
-		(unit 1)
-		(exclude_from_sim no)
-		(in_bom yes)
-		(on_board yes)
-		(dnp no)
-		(fields_autoplaced yes)
-		(property "Reference" "#PWR058"
-			(at 125.73 180.34 0)
-			(effects
-				(font
-					(size 1.27 1.27)
-				)
-				(hide yes)
-			)
-		)
-		(property "Value" "+3V3"
-			(at 125.73 189.23 0)
-			(effects
-				(font
-					(size 1.27 1.27)
-				)
-			)
-		)
-		(property "Footprint" ""
-			(at 125.73 184.15 0)
-			(effects
-				(font
-					(size 1.27 1.27)
-				)
-				(hide yes)
-			)
-		)
-		(property "Datasheet" ""
-			(at 125.73 184.15 0)
-			(effects
-				(font
-					(size 1.27 1.27)
-				)
-				(hide yes)
-			)
-		)
-		(property "Description" "Power symbol creates a global label with name \"+3V3\""
-			(at 125.73 184.15 0)
-			(effects
-				(font
-					(size 1.27 1.27)
-				)
-				(hide yes)
-			)
-		)
-		(pin "1"
-		)
-		(instances
-			(project "DIYDSPv0.8"
-				(path "/b7ce3e82-c245-4515-bd69-0cf398c79f59"
-					(reference "#PWR058")
-					(unit 1)
-				)
-			)
-		)
-	)
-	(symbol
 		(lib_id "Device:R")
 		(at 402.59 267.97 270)
@@
 					(unit 1)
 				)
+			)
+		)
+	)
+	(symbol
+		(lib_id "power:GND")
+		(at 125.73 184.15 0)
+		(unit 1)
+		(exclude_from_sim no)
+		(in_bom yes)
+		(on_board yes)
+		(dnp no)
+		(fields_autoplaced yes)
+		(property "Reference" "#PWR058"
+			(at 125.73 190.5 0)
+			(effects
+				(font
+					(size 1.27 1.27)
+				)
+				(hide yes)
+			)
+		)
+		(property "Value" "GND"
+			(at 125.73 189.23 0)
+			(effects
+				(font
+					(size 1.27 1.27)
+				)
+			)
+		)
+		(property "Footprint" ""
+			(at 125.73 184.15 0)
+			(effects
+				(font
+					(size 1.27 1.27)
+				)
+				(hide yes)
+			)
+		)
+		(property "Datasheet" ""
+			(at 125.73 184.15 0)
+			(effects
+				(font
+					(size 1.27 1.27)
+				)
+				(hide yes)
+			)
+		)
+		(property "Description" "Power symbol creates a global label with name \"GND\" , ground"
+			(at 125.73 184.15 0)
+			(effects
+				(font
+					(size 1.27 1.27)
+				)
+				(hide yes)
+			)
+		)
+		(pin "1"
+		)
+		(instances
+			(project "DIYDSPv0.8"
+				(path "/b7ce3e82-c245-4515-bd69-0cf398c79f59"
+					(reference "#PWR058")
+					(unit 1)
+				)
