File: PCB/DIYDSPv0.8/DIYDSPv0.8.kicad_sch (KiCad schematic)
At the start: 260 parts, among them J1 Conn_01x06, J10 Conn_01x05, J11 Conn_01x05, J12 Conn_01x05, J13 Conn_01x05, J2 Conn_01x05, J3 Conn_01x04, J4 Conn_01x04, J5 Conn_01x02, J6 Conn_01x05, J7 Conn_01x05, J8 Conn_01x05, J9 Conn_01x05, U1 ADAU1452, U4 AMS1117-1.2, X1 12.288MHz

Commit message: Officially ordered v0.8 for validation - 12V input swapped for USB
Parts:
- removed C60: 100n, Capacitor_SMD:C_0402_1005Metric, symbol Device:C
- removed C61: 22u, Capacitor_SMD:C_0805_2012Metric, symbol Device:C
- removed C68: 220uF, Custom:RVT1V221M0810, symbol Custom_Symbol:RVT1V221M0810_C18221522
- removed CN1: ~, Custom:MX126-5.0-02P-GN01-Cu-S-A, symbol Custom_Symbol:MX126-5.0-GN01-02P-CU-S-A
- removed TP3: TestPoint, TestPoint:TestPoint_THTPad_D2.0mm_Drill1.0mm, symbol Connector:TestPoint
- removed U23, U26: ~, Custom:K7803-1000_C50396471, symbol Custom_Symbol:K7803-1000_C50396471
- added D10, D9: ~, Custom:DDZ5V6CSF-7, symbol Custom_Symbol:DDZ5V6CSF-7
- added J14: Conn_01x04, Connector_PinHeader_2.54mm:PinHeader_1x04_P2.54mm_Vertical, symbol Connector_Generic:Conn_01x04
- added R82, R83: 0.2, Resistor_SMD:R_2512_6332Metric, symbol Device:R
- added R84, R85: 5.1k, Resistor_SMD:R_0402_1005Metric, symbol Device:R
- added TP8: TestPoint, TestPoint:TestPoint_THTPad_D2.0mm_Drill1.0mm, symbol Connector:TestPoint
- added U23, U27: ~, Custom:SGM2039A-3.3XXEV8G_TR, symbol Custom_Symbol:SGM2039A-3.3XXEV8G/TR
- added U26: ~, Custom:GT-USB-7010ASV, symbol GT-USB-7010ASV:GT-USB-7010ASV
- C100, C107, C83: value 220uF -> 220u
Connections:
- net +3.3VA: now also R83.2; no longer C111.1
- net +3V3: now also U27.1 (OUT), U27.2 (OUT), U27.4 (FB)
- net GND: now also D10.2 (A), D9.2 (A), J14.1 (Pin_1), J14.2 (Pin_2), R84.1, R85.2, U23.5 (GND), U23.9 (EP), U26.1 (SHELL), U26.2 (SHELL), U26.3 (SHELL), U26.4 (SHELL), U26.A1B12 (GND), U26.B1A12 (GND), U27.5 (GND), U27.9 (EP)
- net VCC: now also D3.1 (C), D9.1 (K), R82.1, TP8.1, U27.6 (EN), U27.7 (IN), U27.8 (IN); no longer C100.1, C110.1, C94.2, C95.2, TP5.1
- net VBUS2: now reaches D3.2 (A)
- net VBUS2: now also U26.A4B9 (VBUS), U26.B4A9 (VBUS)
- net +12V renamed VBUS3
- net VBUS3: now also J14.3 (Pin_3), J14.4 (Pin_4); no longer D3.1 (C)
- new net: R84.2, U26.A5 (CC1)
- new net: R85.1, U26.B5 (CC2)
- new net: C111.1, R83.1, U23.1 (OUT), U23.2 (OUT), U23.4 (FB)
- new net VDD: C100.1, C110.1, C94.2, C95.2, D10.1 (K), R82.2, TP5.1, U23.6 (EN), U23.7 (IN), U23.8 (IN)
- no-connect marks 54 -> 62
Other:
- note added: "Auxilliary connectors for Power"
- moved on the sheet: C103, C104, C107, C110, C111, C116, D7, D8, R68, R69, R74, R75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
