File: PCB/MCL-DSP8x8_OUTPUT_RCA_8/MCL-DSP8x8_OUTPUT_RCA_8.kicad_sch (KiCad schematic)
At the start: 32 parts, among them J1 Conn_01x05, J2 Conn_01x05, J3 Conn_01x05, J4 Conn_01x05

Commit message: Finished design of v1 connector boards.
Parts:
- removed R1, R13, R15, R17, R19, R3, R5, R7: 82k, Resistor_SMD:R_0805_2012Metric_Pad1.20x1.40mm_HandSolder, symbol Device:R
- removed R14, R16, R18, R2, R20, R4, R6, R8: 10k, Resistor_SMD:R_0805_2012Metric_Pad1.20x1.40mm_HandSolder, symbol Device:R
- renumbered R11 to R1, R12 to R2, R21 to R3, R22 to R4, R23 to R5, R9 to R6, R24 to R7, R10 to R8
Connections:
- net RCA_A1+ is gone; now on net A1+: CN1.3
- net RCA_A2+ is gone; now on net A2+: CN1.1
- net RCA_B1+ is gone; now on net B1+: CN2.3
- net RCA_B2+ is gone; now on net B2+: CN2.1
- net RCA_C1+ is gone; now on net C1+: CN3.3
- net RCA_C2+ is gone; now on net C2+: CN3.1
- net RCA_D1+ is gone; now on net D1+: CN4.3
- net RCA_D2+ is gone; now on net D2+: CN4.1
